Commit message: fix the coordinate problem

File: airexo/urdf_models/robot/gripper.urdf (robot description, URDF)
Before this commit: robot gripper, 5 links, 4 joints
Links:
- link gripper_Link1: geometry collision mesh filename=meshes/gripper/Link1.STL; visual mesh filename=meshes/gripper/Link1.STL

File: airexo/urdf_models/robot/true_robot.urdf (robot description, URDF)
Before this commit: robot overseas_75_b_v_description, 45 links, 44 joints
Links:
- link l_gripper_Link1: geometry collision mesh filename=meshes/gripper/Link1.STL; visual mesh filename=meshes/gripper/Link1.STL
- link r_gripper_Link1: geometry collision mesh filename=meshes/gripper/Link1.STL; visual mesh filename=meshes/gripper/Link1.STL
